File: arduino/schematics/countercat_rev2.sch (EAGLE design)
At the start: 32 parts, among them Q1 2N3904, Q2 IRF520, U2 74HC04_HEX_INVERTER, U3 USD-SOCKETNEW, U4 ATMEGA328P_PDIP, Y1 16MHz

Commit message: Slight change.
Parts:
- R6: value (none) -> 10k
Changed lines of the file:
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@@
 <part name="U$5" library="nick_DC2011" deviceset="5V" device=""/>
 <part name="GND5" library="nick_DC2011" deviceset="GND" device=""/>
-<part name="R6" library="SparkFun-Resistors" deviceset="RESISTOR" device="PTH-1/4W"/>
+<part name="R6" library="SparkFun-Resistors" deviceset="RESISTOR" device="PTH-1/4W" value="10k"/>
 <part name="GND6" library="nick_DC2011" deviceset="GND" device=""/>
 <part name="U$6" library="nick_DC2011" deviceset="5V" device=""/>
