File: schematics/countercat_current.brd (EAGLE design)
At the start: 64.8 x 76.2 mm, 59 parts, among them Q1 IRF520, Q3 IRF520, Q4 IRF520, Q5 IRF520, U4 ATMEGA328P, Y1 16MHz

Commit message: Updated current schematic file to fix mistakes from Rev3 board.
Connections:
- removed net N$8: C3.1, U4.20, U4.21, U4.7
- net 5V: now also C3.1, U4.20, U4.21, U4.7; no longer U$7.4, U$7.5
- net GND: now also U$7.4, U$7.5
Routing:
- net N$8: track 25.4 -> 0.00 mm, vias 1 -> 0
- net 5V: track 276.3 -> 288.8 mm, vias 3 -> 4
- net GND: track 238.4 -> 240.9 mm
Other:
- board text added: "5v"
- board text removed: "D7"
Changed lines of the file:
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@@
 <text x="3.81" y="15.875" size="1.016" layer="21" font="fixed">CS</text>
 <text x="3.81" y="23.495" size="1.016" layer="21" font="fixed">SCLK</text>
-<text x="3.81" y="8.255" size="1.016" layer="21" font="fixed">D7</text>
+<text x="3.81" y="8.255" size="1.016" layer="21" font="fixed">5v</text>
 <text x="3.81" y="10.795" size="1.016" layer="21" font="fixed">B0</text>
 <text x="3.81" y="13.335" size="1.016" layer="21" font="fixed">B1</text>
@@
 <contactref element="U$7" pad="16"/>
 <contactref element="C4" pad="1"/>
-<contactref element="U$7" pad="5"/>
-<contactref element="U$7" pad="4"/>
 <contactref element="JP35" pad="2"/>
 <contactref element="JP15" pad="1"/>
-<wire x1="20.32" y1="65.405" x2="17.78" y2="65.405" width="0.2032" layer="1"/>
 <wire x1="33.655" y1="63.5" x2="27.94" y2="57.785" width="0.2032" layer="16"/>
 <wire x1="6.985" y1="13.335" x2="2.54" y2="8.89" width="0.2032" layer="16"/>
@@
 <wire x1="2.54" y1="8.89" x2="2.032" y2="8.89" width="0.2032" layer="16"/>
 <wire x1="56.515" y1="41.275" x2="61.595" y2="41.275" width="0.2032" layer="1"/>
-<wire x1="22.225" y1="63.5" x2="20.32" y2="65.405" width="0.2032" layer="16"/>
 <wire x1="31.115" y1="63.5" x2="22.225" y2="63.5" width="0.2032" layer="16"/>
 <wire x1="8.89" y1="71.755" x2="8.89" y2="69.85" width="0.3048" layer="1"/>
@@
 <wire x1="7.62" y1="61.595" x2="24.13" y2="61.595" width="0.3048" layer="16"/>
 <wire x1="24.13" y1="61.595" x2="27.94" y2="57.785" width="0.3048" layer="16"/>
-<wire x1="20.32" y1="65.405" x2="20.32" y2="73.025" width="0.2032" layer="1"/>
+<contactref element="U4" pad="7"/>
+<contactref element="U4" pad="20"/>
+<contactref element="U4" pad="21"/>
+<contactref element="C3" pad="1"/>
+<wire x1="26.67" y1="34.29" x2="26.67" y2="31.75" width="0.254" layer="1"/>
+<wire x1="24.13" y1="36.83" x2="26.67" y2="34.29" width="0.254" layer="1"/>
+<wire x1="24.13" y1="39.37" x2="24.13" y2="36.83" width="0.254" layer="1"/>
+<wire x1="22.86" y1="40.64" x2="24.13" y2="39.37" width="0.254" layer="16"/>
+<wire x1="15.24" y1="40.64" x2="22.86" y2="40.64" width="0.254" layer="16"/>
+<via x="24.13" y="39.37" extent="1-16" drill="0.6096"/>
+<wire x1="15.24" y1="40.64" x2="15.24" y2="40.005" width="1.016" layer="16"/>
+<wire x1="15.24" y1="40.005" x2="18.415" y2="36.83" width="1.016" layer="16"/>
+<wire x1="18.415" y1="36.83" x2="19.05" y2="36.83" width="1.016" layer="16"/>
+<wire x1="13.97" y1="41.275" x2="14.605" y2="41.275" width="1.016" layer="16"/>
+<wire x1="14.605" y1="41.275" x2="15.24" y2="40.64" width="1.016" layer="16"/>
+<wire x1="29.21" y1="73.025" x2="20.32" y2="73.025" width="0" layer="19" extent="1-1"/>
+<wire x1="24.13" y1="39.37" x2="34.925" y2="42.545" width="0" layer="19" extent="1-1"/>
 </signal>
 <signal name="GND">
@@
 <wire x1="49.53" y1="31.75" x2="61.595" y2="43.815" width="0.254" layer="16"/>
 <wire x1="19.05" y1="3.175" x2="19.05" y2="8.89" width="1.4224" layer="1"/>
+<contactref element="U$7" pad="5"/>
+<contactref element="U$7" pad="4"/>
+<wire x1="20.32" y1="65.405" x2="17.78" y2="65.405" width="0.2032" layer="1"/>
+<wire x1="13.97" y1="71.755" x2="17.78" y2="65.405" width="0" layer="19" extent="16-16"/>
 </signal>
 <signal name="RED">
@@
 <wire x1="13.97" y1="29.21" x2="19.05" y2="29.21" width="1.016" layer="1"/>
 </signal>
-<signal name="N$8">
-<contactref element="U4" pad="7"/>
-<contactref element="U4" pad="20"/>
-<contactref element="U4" pad="21"/>
-<contactref element="C3" pad="1"/>
-<wire x1="26.67" y1="34.29" x2="26.67" y2="31.75" width="0.254" layer="1"/>
-<wire x1="24.13" y1="36.83" x2="26.67" y2="34.29" width="0.254" layer="1"/>
-<wire x1="24.13" y1="39.37" x2="24.13" y2="36.83" width="0.254" layer="1"/>
-<wire x1="22.86" y1="40.64" x2="24.13" y2="39.37" width="0.254" layer="16"/>
-<wire x1="15.24" y1="40.64" x2="22.86" y2="40.64" width="0.254" layer="16"/>
-<via x="24.13" y="39.37" extent="1-16" drill="0.6096"/>
-<wire x1="15.24" y1="40.64" x2="15.24" y2="40.005" width="1.016" layer="16"/>
-<wire x1="15.24" y1="40.005" x2="18.415" y2="36.83" width="1.016" layer="16"/>
-<wire x1="18.415" y1="36.83" x2="19.05" y2="36.83" width="1.016" layer="16"/>
-<wire x1="13.97" y1="41.275" x2="14.605" y2="41.275" width="1.016" layer="16"/>
-<wire x1="14.605" y1="41.275" x2="15.24" y2="40.64" width="1.016" layer="16"/>
-</signal>
 <signal name="PUSH">
